Commit message: added sfb tail

File: robot_assets/RSRR_tail/rsrr_urdf.urdf (robot description, URDF)
Before this commit: robot rsu_urdf, 9 links, 8 joints
Links:
- link base_link: mass 0.020099668041423 -> 0.0201
- link left_mid: mass 0.00772015470242627 -> 0.0077202
- link left_rod: mass 0.0154173178374304 -> 0.015417
- link main_mid: mass 0.0169792722258016 -> 0.016979
- link main_rod: mass 0.251856293416819 -> 0.25186
- link motor_left: mass 0.00429498890692695 -> 0.004295
- link motor_right: mass 0.00429498885337272 -> 0.004295
- link right_mid: mass 0.00772015470242627 -> 0.0077202
- link right_rod: mass 0.0165482911927227 -> 0.016548
Joints:
- removed joint alpha
- added joint alpha1: type revolute, parent base_link, child main_mid, origin xyz=0 0 0 rpy=0 0 0, axis 0 1 0, limit lower=-1.5707 upper=1.5707
- joint alpha2: limit lower=-1.5707 upper=1.5707 effort=0 velocity=0 -> lower=-1.5707 upper=1.5707; origin xyz=-0.014963 0.0010507 -0.0105 rpy=1.5708 0 -1.6409 -> xyz=0 0 0.015 rpy=0 0 0
- joint phi1: limit lower=-1.5707 upper=1.5707 effort=0 velocity=0 -> lower=-1.5707 upper=1.5707; origin xyz=-0.02 0 0.03 rpy=1.5708 0 0 -> xyz=-0.02 0.03 0 rpy=0 0 0
- joint phi2: axis -1 0 0 -> 1 0 0; limit lower=-1.5707 upper=1.5707 effort=0 velocity=0 -> lower=-1.5707 upper=1.5707
- joint psi1: limit lower=-1.5707 upper=1.5707 effort=0 velocity=0 -> lower=-1.5707 upper=1.5707; origin xyz=0.02 0 0.03 rpy=1.5708 0 0 -> xyz=0.02 0.03 0 rpy=0 0 0
- joint psi2: axis -1 0 0 -> 1 0 0; limit lower=0 upper=1.5707 effort=0 velocity=0 -> lower=-1.5707 upper=1.5707
- joint theta1: limit lower=-1.5707 upper=1.5707 effort=0 velocity=0 -> lower=-1.5707 upper=1.5707
- joint theta2: axis -1 0 0 -> 1 0 0; limit lower=-1.5707 upper=1.5707 effort=0 velocity=0 -> lower=-1.5707 upper=1.5707
